Commit message: update  gazebo sim sensors and robot

File: src/aibee_robot/config/vr_bot.xacro (robot description, xacro)
@@ -1,2 +1,3 @@
+<?xml version="1.0"?>
 <!--
   Copyright 2016 The Cartographer Authors
@@ -12,5 +13,5 @@
 -->
 <!-- robot -->
-<robot name="aibee_robot">
+<robot name="aibee_robot" xmlns:xacro="http://ros.org/wiki/xacro">
   <material name="orange">
     <color rgba="1.0 0.5 0.2 1" />
@@ -59,12 +60,4 @@
     </visual>
   </link>
-    <link name="${pos}_sonar">
-      <visual>
-        <origin xyz="0 0 0" rpy="0 1.57 0"/>
-        <geometry>
-          <cylinder length="0.01" radius="0.01"/>
-        </geometry>
-      </visual>
-    </link>
 <!-- odom_child
   <link name="odom_child">
@@ -103,3 +96,4 @@
 <origin xyz="-0.00493858 0.102603 -0.801653" rpy="0.00584294 0.00656523 1.58415" />
   </joint> -->
+  </xacro:macro>
 </robot>

File: src/ros_gazebo_sim/gazebo_robot/robot/mrobot_with_sensors.xacro (robot description, xacro)
@@ -8,4 +8,5 @@
     <xacro:arg name="imu_enabled" default="false" />
     <xacro:arg name="gps_enabled" default="false" />
+    <xacro:arg name="mulit_sonars_enabled" default="false" />
     <xacro:property name="M_PI" value="3.14159"/>
     <xacro:arg name="robot_namespace" default="/" />
@@ -45,7 +46,7 @@
         <xacro:sick_lms1xx_mount prefix="base" />
         <sick_lms1xx frame="base_laser" topic="scan" robot_namespace="$(arg robot_namespace)"/>
-        <xacro:property name="sick_offset_x" value="0.1" />
+        <xacro:property name="sick_offset_x" value="0" />
         <xacro:property name="sick_offset_y" value="0" />
-        <xacro:property name="sick_offset_z" value="0.02" />
+        <xacro:property name="sick_offset_z" value="0.001" />
         <!-- sick_lms1xx_enabled-joint -->
         <joint name="sick_lms1xx_joint" type="fixed">
@@ -61,5 +62,5 @@
         <xacro:property name="imu_offset_x" value="0" />
         <xacro:property name="imu_offset_y" value="0" />
-        <xacro:property name="imu_offset_z" value="0.02" />
+        <xacro:property name="imu_offset_z" value="0.001" />
         <!-- imu_link-joint -->
         <joint name="imu_link_joint" type="fixed">
@@ -73,11 +74,11 @@
         <xacro:include filename="$(find gazebo_robot)/sensors/gps/urdf/gps.xacro"/>
         <xacro:gps  robot_namespace="$(arg robot_namespace)"/>
-        <xacro:property name="gps_offset_x" value="0.1" />
-        <xacro:property name="gps_offset_y" value="0.1" />
-        <xacro:property name="gps_offset_z" value="0.02" />
+        <xacro:property name="gps_offset_x" value="0" />
+        <xacro:property name="gps_offset_y" value="0" />
+        <xacro:property name="gps_offset_z" value="0.001" />
         <!-- gps_link-joint -->
         <joint name="gps_link_joint" type="fixed">
             <origin xyz="${gps_offset_x} ${gps_offset_y} ${gps_offset_z}" rpy="0 0 0" />
-            <parent link="plate_1_link"/>
+            <parent link="base_link"/>
             <child link="gps_link"/>
         </joint>
@@ -107,3 +108,18 @@
         </HDL-32E>
     </xacro:if> <!-- velodyne32_enabled -->
+    <!-- mulit_sonars_enabled module  ============================================================================================= -->
+    <xacro:if value="$(arg mulit_sonars_enabled)">
+    <!-- s1_front -->
+    <xacro:include filename="$(find gazebo_robot)/sensors/sonar/urdf/sonar.xacro"/>
+    <xacro:sonar parent="plate_2_link" pos="s1" xyz="0.12 0 0.02 " rpy="0 -3.1415 3.1415" />
+    <!-- s2_front left -->
+    <xacro:include filename="$(find gazebo_robot)/sensors/sonar/urdf/sonar.xacro"/>
+    <xacro:sonar parent="plate_2_link" pos="s2" xyz="0.12 0.04 0.02 " rpy="0 -3.1415 -2.094" />
+    <!-- s2_front right -->
+    <xacro:include filename="$(find gazebo_robot)/sensors/sonar/urdf/sonar.xacro"/>
+    <xacro:sonar parent="plate_2_link" pos="s3" xyz="0.12 -0.04 0.02 " rpy="0 -3.1415 2.094" />
+    <!-- back -->
+    <xacro:include filename="$(find gazebo_robot)/sensors/sonar/urdf/sonar.xacro"/>
+    <xacro:sonar parent="plate_2_link" pos="s4" xyz="-0.12 0 0.02 " rpy="0 -3.1415 0" />
+    </xacro:if> <!-- mulit-sonars_enabled  -->
 </robot>

File: src/ros_gazebo_sim/gazebo_robot/sensors/gps/urdf/gps.xacro (robot description, xacro)
@@ -15,5 +15,5 @@
     <inertial>
       <origin xyz="0 0 0"/>
-      <mass value="1"/>
+      <mass value="0.01"/>
       <inertia ixx="3.0" ixy="0.0" ixz="0.0"
                iyy="3.0" iyz="0.0"

File: src/ros_gazebo_sim/gazebo_robot/sensors/mrobot/urdf/mrobot_body.urdf.xacro (robot description, xacro)
@@ -18,5 +18,5 @@
     <xacro:property name="M_PI" value="3.1415926535897931" />
     <!-- Main body length, width, height and mass -->
-    <xacro:property name="base_mass"        value="0.5" />
+    <xacro:property name="base_mass"        value="1.50" /> <!-- mass origin  0.5-->
     <xacro:property name="base_link_radius" value="0.13"/>
     <xacro:property name="base_link_length" value="0.005"/>
@@ -24,12 +24,12 @@
     <!-- Caster radius and mass -->
     <xacro:property name="caster_radius"          value="0.016" />
-    <xacro:property name="caster_mass"            value="0.01" />
+    <xacro:property name="caster_mass"            value="0.1" /> <!-- mass origin 0.01-->
     <xacro:property name="caster_joint_origin_x"  value="-0.12" />
     <!-- Wheel radius, height and mass -->
     <xacro:property name="wheel_radius" value="0.033" />
     <xacro:property name="wheel_height" value="0.017" />
-    <xacro:property name="wheel_mass"   value="0.1" />
+    <xacro:property name="wheel_mass"   value="0.10" /> <!-- mass origin 0.1-->
     <!-- plate height and mass -->
-    <xacro:property name="plate_mass"   value="0.05"/>
+    <xacro:property name="plate_mass"   value="0.5"/><!-- mass origin 0.05-->
     <xacro:property name="plate_height" value="0.07"/>
     <xacro:property name="standoff_x"   value="0.12"/>

File: src/ros_gazebo_sim/gazebo_robot/sensors/sonar/urdf/sonar.xacro (robot description, xacro)
@@ -18,9 +18,9 @@
       </collision>
     </link>
-    <!-- <joint name="${pos}_sonar_joint" type="fixed">
+    <joint name="${pos}_sonar_joint" type="fixed">
         <origin xyz="${xyz}" rpy="${rpy}"/>
         <parent link="${parent}"/>
         <child link="${pos}_sonar"/>
-    </joint> -->
+    </joint>
     <gazebo reference="${pos}_sonar">
       <sensor type="ray" name="sonar">

File: src/ros_gazebo_sim/gazebo_robot/sensors/usb_camera/urdf/usb_camera.xacro (robot description, xacro)
@@ -4,5 +4,5 @@
         <link name="${prefix}_link">
             <inertial>
-                <mass value="0.1" />
+                <mass value="0.01" />
                 <origin xyz="0 0 0" />
                 <inertia ixx="0.01" ixy="0.0" ixz="0.0"

File: src/ros_gazebo_sim/gazebo_robot/sensors/velodyne/urdf/HDL-32E.urdf.xacro (robot description, xacro)
@@ -12,5 +12,5 @@
     <link name="${name}_base_link">
       <inertial>
-        <mass value="1.0"/>
+        <mass value="0.010"/>
         <origin xyz="0 0 0.07212"/>
         <inertia ixx="${(1.0 * (3.0*0.04267*0.04267 + 0.14424*0.14424)) / 12.0}" ixy="0" ixz="0"
@@ -38,5 +38,5 @@
     <link name="${name}">
       <inertial>
-        <mass value="0.01"/>
+        <mass value="0.001"/>
         <origin xyz="0 0 0"/>
         <inertia ixx="1e-7" ixy="0" ixz="0" iyy="1e-7" iyz="0" izz="1e-7"/>

File: src/ros_gazebo_sim/gazebo_robot/sensors/velodyne/urdf/VLP-16.urdf.xacro (robot description, xacro)
@@ -10,5 +10,5 @@
     <link name="${name}_base_link">
       <inertial>
-        <mass value="0.83"/>
+        <mass value="0.03"/>
         <origin xyz="0 0 0.03585"/>
         <inertia ixx="${(0.83 * (3.0*0.0516*0.0516 + 0.0717*0.0717)) / 12.0}" ixy="0" ixz="0"

File: src/ros_gazebo_sim/mrobot_description/urdf/mrobot_body.urdf.xacro (robot description, xacro)
@@ -263,4 +263,7 @@
             </plugin>
         </gazebo>
+    <!-- s1_front -->
+    <xacro:include filename="$(find gazebo_robot)/sensors/sonar/urdf/sonar.xacro"/>
+    <xacro:sonar parent="plate_2_link" pos="s1" xyz="0.12 0 0.02 " rpy="0 -3.1415 3.1415" />
     </xacro:macro>
 </robot>

Commit message: update vr_bot.xacro

File: src/aibee_robot/config/vr_bot.xacro (robot description, xacro)
@@ -50,14 +50,38 @@
     </visual>
   </link>
-<!-- vertical_vlp16_link  -->
-  <link name="vertical_vlp16_link">
-    <visual>
-      <origin xyz="0.0 0.0 0.0" />
-      <geometry>
-        <cylinder length="0.07" radius="0.05" />
-      </geometry>
-      <material name="gray" />
-    </visual>
-  </link>
+<!-- sonars sensor -->
+  <!-- UM6-IMU -->
+  <xacro:include filename="$(find aibee_robot)/config/sonar.xacro"/>
+  <xacro:sonar parent="base_link" pos="m1" xyz="-0.3402  0.1611 0.0497 " rpy="0 1.57 0" />
+  <xacro:include filename="$(find aibee_robot)/config/sonar.xacro"/>
+  <xacro:sonar parent="base_link" pos="m2" xyz="-0.1276 0.2838 0.0497 " rpy="0 1.57 0" />
+  <xacro:include filename="$(find aibee_robot)/config/sonar.xacro"/>
+  <xacro:sonar parent="base_link" pos="m3" xyz="0.05 0.2693 0.0497 " rpy="0 1.57 0" />
+  <xacro:include filename="$(find aibee_robot)/config/sonar.xacro"/>
+  <xacro:sonar parent="base_link" pos="m4" xyz="0.1514 0.1227 0.0497 " rpy="0 1.57 0" />
+  <xacro:include filename="$(find aibee_robot)/config/sonar.xacro"/>
+  <xacro:sonar parent="base_link" pos="m5" xyz="0.1514 -0.1227 0.0497 " rpy="0 1.57 0" />
+  <xacro:include filename="$(find aibee_robot)/config/sonar.xacro"/>
+  <xacro:sonar parent="base_link" pos="m6" xyz="0.05 -0.2693 0.0497 " rpy="0 1.57 0" />
+  <xacro:include filename="$(find aibee_robot)/config/sonar.xacro"/>
+  <xacro:sonar parent="base_link" pos="m7" xyz="-0.1276 -0.2838 0.0497 " rpy="0 1.57 0" />
+  <xacro:include filename="$(find aibee_robot)/config/sonar.xacro"/>
+  <xacro:sonar parent="base_link" pos="m8" xyz="-0.3402  -0.1611 0.0497" rpy="0 1.57 0" />
+  <xacro:include filename="$(find aibee_robot)/config/sonar.xacro"/>
+  <xacro:sonar parent="base_link" pos="m9" xyz="0 0 0 " rpy="0 1.57 0" />
+<!-- rplidar sensor  -->
+    <link name="rplidar_link">
+      <visual>
+        <origin xyz="0 0 0" rpy="0 1.57 0"/>
+        <geometry>
+          <cylinder length="0.05" radius="0.05"/>
+        </geometry>
+      </visual>
+    </link>
+    <joint name="rplidar_link_joint" type="fixed">
+        <origin xyz="0.1127 0 0.013" rpy="0 1.57 0"/>
+        <parent link="base_link"/>
+        <child link="rplidar_link"/>
+    </joint>
 <!-- odom_child
   <link name="odom_child">

File: src/ros_gazebo_sim/gazebo_robot/robot/test_sonar.xacro (robot description, xacro)
@@ -30,9 +30,4 @@
     </inertial>
   </link>
-    <joint name="sonar_frame_joint" type="fixed">
-      <parent link="base_link"/>
-      <child link="m1_sonar"/>
-      <origin xyz="0 0 0.8" rpy="0 0 -3.14" />
-    </joint>
   <!-- UM6-IMU -->
   <xacro:include filename="$(find gazebo_robot)/sensors/sonar/urdf/sonar.xacro"/>
