Commit message: update

File: src/aibee_robot/config/vr_bot.1.xacro (robot description, xacro)
@@ -11,6 +11,8 @@
   limitations under the License.
 -->
+<?xml version="1.0"?>
+<robot name="aibee_robot" xmlns:xacro="http://ros.org/wiki/xacro">
+  <xacro:macro name="aibee_robot" >
 <!-- robot -->
-<robot name="aibee_robot">
   <material name="orange">
     <color rgba="1.0 0.5 0.2 1" />
@@ -78,40 +80,6 @@
     <parent link="imu_link" />
     <child link="vertical_vlp16_link" />
-    <origin xyz="0.0107642 0.17024 0.0459122" rpy="0.029518 1.31004 1.58561" />
+<origin xyz="0.0107642 0.17024 0.0459122" rpy="0.029518 1.31004 1.58561" />
   </joint>
-<!-- rplidar sensor  -->
-    <link name="rplidar_link">
-      <visual>
-        <origin xyz="0 0 0" rpy="0 1.57 0"/>
-        <geometry>
-          <cylinder length="0.05" radius="0.05"/>
-        </geometry>
-      </visual>
-    </link>
-    <joint name="rplidar_link_joint" type="fixed">
-        <parent link="base_link"/>
-        <child link="rplidar_link"/>
-        <origin xyz="0.1127 0 0.013" rpy="0 1.57 0"/>
-    </joint>
-<!-- sonars sensor -->
-  <!-- UM6-IMU -->
-  <xacro:include filename="$(find aibee_robot)/config/sonar.xacro"/>
-  <xacro:sonar parent="base_link" pos="m1" xyz="-0.3402  0.1611 0.0497 " rpy="0 1.57 0" />
-  <xacro:include filename="$(find aibee_robot)/config/sonar.xacro"/>
-  <xacro:sonar parent="base_link" pos="m2" xyz="-0.1276 0.2838 0.0497 " rpy="0 1.57 0" />
-  <xacro:include filename="$(find aibee_robot)/config/sonar.xacro"/>
-  <xacro:sonar parent="base_link" pos="m3" xyz="0.05 0.2693 0.0497 " rpy="0 1.57 0" />
-  <xacro:include filename="$(find aibee_robot)/config/sonar.xacro"/>
-  <xacro:sonar parent="base_link" pos="m4" xyz="0.1514 0.1227 0.0497 " rpy="0 1.57 0" />
-  <xacro:include filename="$(find aibee_robot)/config/sonar.xacro"/>
-  <xacro:sonar parent="base_link" pos="m5" xyz="0.1514 -0.1227 0.0497 " rpy="0 1.57 0" />
-  <xacro:include filename="$(find aibee_robot)/config/sonar.xacro"/>
-  <xacro:sonar parent="base_link" pos="m6" xyz="0.05 -0.2693 0.0497 " rpy="0 1.57 0" />
-  <xacro:include filename="$(find aibee_robot)/config/sonar.xacro"/>
-  <xacro:sonar parent="base_link" pos="m7" xyz="-0.1276 -0.2838 0.0497 " rpy="0 1.57 0" />
-  <xacro:include filename="$(find aibee_robot)/config/sonar.xacro"/>
-  <xacro:sonar parent="base_link" pos="m8" xyz="-0.3402  -0.1611 0.0497" rpy="0 1.57 0" />
-  <xacro:include filename="$(find aibee_robot)/config/sonar.xacro"/>
-  <xacro:sonar parent="base_link" pos="m9" xyz="0 0 0 " rpy="0 1.57 0" />
   <!-- <joint name="odom_child_joint" type="fixed">
     <parent link="base_link" />
@@ -119,3 +87,4 @@
 <origin xyz="-0.00493858 0.102603 -0.801653" rpy="0.00584294 0.00656523 1.58415" />
   </joint> -->
+  </xacro:macro>
 </robot>

File: src/aibee_robot/config/vr_bot.xacro (robot description, xacro)
@@ -14,8 +14,9 @@
 <!-- robot -->
 <robot name="aibee_robot" xmlns:xacro="http://ros.org/wiki/xacro">
+  <xacro:macro name="aibee_robot" >
   <material name="orange">
     <color rgba="1.0 0.5 0.2 1" />
-  </material>
-  <material name="gray">
+      </material>
+      <material name="gray">
     <color rgba="0.2 0.2 0.2 1" />
   </material>
@@ -50,4 +51,6 @@
     </visual>
   </link>
+  <!--base_link -->
+  <link name="base_link" />
 <!-- sonars sensor -->
   <!-- UM6-IMU -->
@@ -80,20 +83,8 @@
     </link>
     <joint name="rplidar_link_joint" type="fixed">
-        <origin xyz="0.1127 0 0.013" rpy="0 1.57 0"/>
         <parent link="base_link"/>
         <child link="rplidar_link"/>
+        <origin xyz="0.1127 0 0.013" rpy="0 1.57 0"/>
     </joint>
-<!-- odom_child
-  <link name="odom_child">
-    <visual>
-      <origin xyz="0.0 0.0 0.0" />
-      <geometry>
-        <box size="0.06 0.04 0.02" />
-      </geometry>
-      <material name="orange" />
-    </visual>
-  </link> -->
-  <!--base_link -->
-  <link name="base_link" />
 <!-- the joint of every link -->
 <!-- base_link ==> imu -->
@@ -113,11 +104,6 @@
     <parent link="imu_link" />
     <child link="vertical_vlp16_link" />
-<origin xyz="0.0107642 0.17024 0.0459122" rpy="0.029518 1.31004 1.58561" />
+    <origin xyz="0.0107642 0.17024 0.0459122" rpy="0.029518 1.31004 1.58561" />
   </joint>
-  <!-- <joint name="odom_child_joint" type="fixed">
-    <parent link="base_link" />
-    <child link="odom_child" />
-<origin xyz="-0.00493858 0.102603 -0.801653" rpy="0.00584294 0.00656523 1.58415" />
-  </joint> -->
   </xacro:macro>
 </robot>
