Commit message: update in the robot

File: src/aibee_robot/config/vr_bot.urdf (robot description, URDF)
Before this commit: robot cartographer_backpack_3d, 5 links, 4 joints
Links:
- removed link odom_child
Joints:
- removed joint odom_child_joint
- joint horizontal_vlp16_link_joint: parent base_link -> imu_link
- joint imu_link_joint: origin xyz=0 0 0 rpy=0 0 0 -> xyz=0.00493858 0.00 0.801653 rpy=-0.00584294 -0.00656523 -1.58415
- joint vertical_vlp16_link_joint: parent base_link -> imu_link

Commit message: update

File: src/aibee_robot/config/vr_bot.urdf (robot description, URDF)
Before this commit: robot aibee_robot, 8 links, 7 joints
Links:
- link m1_sonar: geometry visual cylinder length=0.01 radius=0.01
- link m2_sonar: geometry visual cylinder length=0.01 radius=0.01
- link m3_sonar: geometry visual cylinder length=0.01 radius=0.01
Joints:
- joint rplidar_link_joint: origin xyz=0.1127 0 0.013 rpy=0 1.57 0 -> xyz=0.1127 0 0.013 rpy=0 0 0

Commit message: update

File: src/aibee_robot/config/vr_bot.urdf (robot description, URDF)
Before this commit: robot aibee_robot, 8 links, 7 joints
Links:
- added link m4_sonar; visual cylinder length=0.01 radius=0.01
- added link m5_sonar; visual cylinder length=0.01 radius=0.01
- added link m6_sonar; visual cylinder length=0.01 radius=0.01
- added link m7_sonar; visual cylinder length=0.01 radius=0.01
- added link m8_sonar; visual cylinder length=0.01 radius=0.01
- added link m9_sonar; visual cylinder length=0.01 radius=0.01
Joints:
- added joint m4_sonar_joint: type fixed, parent base_link, child m4_sonar, origin xyz=0.1514 0.1227 0.0497  rpy=0 0 0
- added joint m5_sonar_joint: type fixed, parent base_link, child m5_sonar, origin xyz=0.1514 -0.1227 0.0497  rpy=0 0 0
- added joint m6_sonar_joint: type fixed, parent base_link, child m6_sonar, origin xyz=0.05 -0.2693 0.0497  rpy=0 0 0
- added joint m7_sonar_joint: type fixed, parent base_link, child m7_sonar, origin xyz=-0.1276 -0.2838 0.0497  rpy=0 1.57 0
- added joint m8_sonar_joint: type fixed, parent base_link, child m8_sonar, origin xyz=0 0 0  rpy=0 0 -3.1415
- joint m1_sonar_joint: origin xyz=-0.3402  0.1611 0.0497 rpy=0 0 0 -> xyz=-0.3402  0.1611 0.0497 rpy=0 0 0 -2.699
- joint m2_sonar_joint: origin xyz=-0.1276 0.2838 0.0497  rpy=0 1.57 0 -> xyz=-0.1276 0.2838 0.0497  rpy=0 0 0
- joint m3_sonar_joint: origin xyz=0.05 0.2693 0.0497  rpy=0 1.57 0 -> xyz=0.05 0.2693 0.0497  rpy=0 0 0

Commit message: update

File: src/aibee_robot/config/vr_bot.urdf (robot description, URDF)
Before this commit: robot aibee_robot, 14 links, 12 joints
Joints:
- joint m1_sonar_joint: origin xyz=-0.3402  0.1611 0.0497 rpy=0 0 0 -2.699 -> xyz=-0.3402  0.1611 0.0497 rpy=0 0  -2.699

Commit message: update

File: src/aibee_robot/config/vr_bot.urdf (robot description, URDF)
Before this commit: robot aibee_robot, 14 links, 12 joints
Joints:
- added joint m9_sonar_joint: type fixed, parent base_link, child m9_sonar, origin xyz=0 0 0  rpy=0 0 -3.1415
- joint m8_sonar_joint: origin xyz=0 0 0  rpy=0 0 -3.1415 -> xyz=-0.3402  -0.1611 0.0497 rpy=0 0 2.699

Commit message: update

File: src/aibee_robot/config/vr_bot.urdf (robot description, URDF)
Before this commit: robot aibee_robot, 14 links, 13 joints
Joints:
- joint m2_sonar_joint: origin xyz=-0.1276 0.2838 0.0497  rpy=0 0 0 -> xyz=-0.1276 0.2838 0.0497  rpy=0 0 1.9933
- joint m3_sonar_joint: origin xyz=0.05 0.2693 0.0497  rpy=0 0 0 -> xyz=0.05 0.2693 0.0497  rpy=0 0 -1.7544
- joint m6_sonar_joint: origin xyz=0.05 -0.2693 0.0497  rpy=0 0 0 -> xyz=0.05 -0.2693 0.0497  rpy=0 0 -1.7544
- joint m7_sonar_joint: origin xyz=-0.1276 -0.2838 0.0497  rpy=0 1.57 0 -> xyz=-0.1276 -0.2838 0.0497  rpy=0 0 -1.9933
- joint m8_sonar_joint: origin xyz=-0.3402  -0.1611 0.0497 rpy=0 0 2.699 -> xyz=-0.3402  -0.1611 0.0497 rpy=0 0 -2.699
- joint m9_sonar_joint: origin xyz=0 0 0  rpy=0 0 -3.1415 -> xyz=-0.4165 0 0.0497  rpy=0 0 -3.1415

Commit message: update

File: src/aibee_robot/config/vr_bot.urdf (robot description, URDF)
Before this commit: robot aibee_robot, 14 links, 13 joints
Joints:
- joint m1_sonar_joint: origin xyz=-0.3402  0.1611 0.0497 rpy=0 0  -2.699 -> xyz=-0.3402  0.1611 0.0497 rpy=0 0  2.0131
- joint m8_sonar_joint: origin xyz=-0.3402  -0.1611 0.0497 rpy=0 0 -2.699 -> xyz=-0.3402  -0.1611 0.0497 rpy=0 0 -2.0131

Commit message: update

File: src/aibee_robot/config/vr_bot.urdf (robot description, URDF)
Before this commit: robot aibee_robot, 14 links, 13 joints
Joints:
- joint m2_sonar_joint: origin xyz=-0.1276 0.2838 0.0497  rpy=0 0 1.9933 -> xyz=-0.1276 0.2838 0.0497  rpy=0 0 2.719
- joint m7_sonar_joint: origin xyz=-0.1276 -0.2838 0.0497  rpy=0 0 -1.9933 -> xyz=-0.1276 -0.2838 0.0497  rpy=0 0 -2.719

Commit message: add  rplidar  obstacle layer

File: src/aibee_robot/config/vr_bot.urdf (robot description, URDF)
Before this commit: robot aibee_robot, 14 links, 13 joints
Joints:
- joint rplidar_link_joint: origin xyz=0.1127 0 0.013 rpy=0 0 0 -> xyz=0.1127 0  0.013 rpy=0 0 0

Commit message: update

File: src/aibee_robot/config/vr_bot.urdf (robot description, URDF)
Before this commit: robot aibee_robot, 14 links, 13 joints
Joints:
- joint m1_sonar_joint: origin xyz=-0.3402  0.1611 0.0497 rpy=0 0  2.0131 -> xyz=-0.3402  0.1611 0.0497 rpy=0 0  2.2626
- joint m2_sonar_joint: origin xyz=-0.1276 0.2838 0.0497  rpy=0 0 2.719 -> xyz=-0.1276 0.2838 0.0497  rpy=0 0 1.9268
- joint m3_sonar_joint: origin xyz=0.05 0.2693 0.0497  rpy=0 0 -1.7544 -> xyz=0.05 0.2693 0.0497  rpy=0 0 1.0472
- joint m4_sonar_joint: origin xyz=0.1514 0.1227 0.0497  rpy=0 0 0 -> xyz=0.1514 0.1227 0.0497  rpy=0 0 0.1682
- joint m5_sonar_joint: origin xyz=0.1514 -0.1227 0.0497  rpy=0 0 0 -> xyz=0.1514 -0.1227 0.0497  rpy=0 0 -0.1682
- joint m6_sonar_joint: origin xyz=0.05 -0.2693 0.0497  rpy=0 0 -1.7544 -> xyz=0.05 -0.2693 0.0497  rpy=0 0 -1.0472
- joint m7_sonar_joint: origin xyz=-0.1276 -0.2838 0.0497  rpy=0 0 -2.719 -> xyz=-0.1276 -0.2838 0.0497  rpy=0 0 -1.9268
- joint m8_sonar_joint: origin xyz=-0.3402  -0.1611 0.0497 rpy=0 0 -2.0131 -> xyz=-0.3402  -0.1611 0.0497 rpy=0 0 -2.2626

Commit message: update

File: src/aibee_robot/config/vr_bot.urdf (robot description, URDF)
Before this commit: robot aibee_robot, 14 links, 13 joints
Links:
- removed link m9_sonar
- added link m0_sonar; visual cylinder length=0.01 radius=0.01
Joints:
- removed joint m9_sonar_joint
- added joint m0_sonar_joint: type fixed, parent base_link, child m0_sonar, origin xyz=-0.3402  0.1611 0.0497 rpy=0 0  2.2626
- joint m1_sonar_joint: origin xyz=-0.3402  0.1611 0.0497 rpy=0 0  2.2626 -> xyz=-0.1276 0.2838 0.0497  rpy=0 0 1.9268
- joint m2_sonar_joint: origin xyz=-0.1276 0.2838 0.0497  rpy=0 0 1.9268 -> xyz=0.05 0.2693 0.0497  rpy=0 0 1.0472
- joint m3_sonar_joint: origin xyz=0.05 0.2693 0.0497  rpy=0 0 1.0472 -> xyz=0.1514 0.1227 0.0497  rpy=0 0 0.1682
- joint m4_sonar_joint: origin xyz=0.1514 0.1227 0.0497  rpy=0 0 0.1682 -> xyz=0.1514 -0.1227 0.0497  rpy=0 0 -0.1682
- joint m5_sonar_joint: origin xyz=0.1514 -0.1227 0.0497  rpy=0 0 -0.1682 -> xyz=0.05 -0.2693 0.0497  rpy=0 0 -1.0472
- joint m6_sonar_joint: origin xyz=0.05 -0.2693 0.0497  rpy=0 0 -1.0472 -> xyz=-0.1276 -0.2838 0.0497  rpy=0 0 -1.9268
- joint m7_sonar_joint: origin xyz=-0.1276 -0.2838 0.0497  rpy=0 0 -1.9268 -> xyz=-0.3402  -0.1611 0.0497 rpy=0 0 -2.2626
- joint m8_sonar_joint: origin xyz=-0.3402  -0.1611 0.0497 rpy=0 0 -2.2626 -> xyz=-0.4165 0 0.0497  rpy=0 0 -3.1415
